File: PCB/MotoGymkhanaRaceTiming/MotoGymkhanaRaceTiming.kicad_pcb (KiCad board)
At the start: 2 copper layers, 99.1 x 64.8 mm, 42 parts, among them U1 LM2577T-ADJ_NOPB, U2 PC817, U3 PC817

Commit message: Schematic optimizations
Parts:
- LED_FIN1, LED_START1, PWR1: moved to B.Cu
- moved R_SQW1 78.9 mm to (63.5, 72.4)
- moved C1 73.8 mm to (54.6, 40.6)
- moved C2 73.8 mm to (104.1, 87.6)
- moved D1 73.8 mm to (110.5, 61.0)
- moved L1 73.8 mm to (104.1, 49.5)
- moved MCU_1 73.8 mm to (40.6, 67.3)
- moved R1 73.8 mm to (97.8, 31.8)
- moved R33 73.8 mm to (110.5, 76.2)
- moved R39 73.8 mm to (114.3, 66.0)
- moved R_FIN1 73.8 mm to (124.5, 81.3)
- moved R_PD_B1 73.8 mm to (76.2, 55.9)
- moved R_PD_B2 73.8 mm to (94.0, 48.3)
- moved R_PD_Fin1 73.8 mm to (59.7, 58.4)
- moved R_PD_St1 73.8 mm to (54.6, 58.4)
- moved SENS_FIN1 73.8 mm to (125.7, 64.8)
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Connections:
- net Net-(C1-Pad1) renamed +5V
- net Net-(C1-Pad2) renamed GND
- net Net-(C4-Pad1) renamed /12V
Routing:
- net Net-(MCU_1-Pad11): track 19.9 -> 25.7 mm
- net +5V: track 344.4 -> 346.6 mm, vias 0 -> 1
- net Net-(MCU_1-Pad15): track 32.2 -> 33.3 mm
- net Net-(LED_FIN1-Pad2): track 99.9 -> 98.8 mm
Other:
- board text added: "PWR1, LED_S and LED_F on back of board"
